Commit message: update sensor

File: src/semi_humanoid_v2/urdf/gazebo_plugins.xacro (robot description, xacro)
@@ -122,7 +122,9 @@
        sensors are expensive and enabling all of them at once will not
        hold real-time on a Jetson. See gazebo.launch.py arguments
-       lidar_3d / camera / side_cameras.
+       camera / side_cameras / airy / airy_back.
        ══════════════════════════════════════════════════════════════════ -->
-  <!-- ── 3D LiDAR (gpu_lidar, Vanjee WLR-722 approximation) ──
+  <!-- ── Generic 3D LiDAR (gpu_lidar). The stock ANTBot mount is gone, but
+       this macro is what airy_lidar.xacro builds each RoboSense Airy from, so
+       its lidar_3d_* parameter defaults are only defaults. ──
        Fortress gpu_lidar publishes TWO topics:
          <topic>          ignition.msgs.LaserScan

File: src/semi_humanoid_v2/urdf/semi_humanoid_v2_airy.urdf.xacro (robot description, xacro)
@@ -1,43 +1,77 @@
 <?xml version="1.0" ?>
 <!--
-  semi_humanoid_v2_real.urdf.xacro + two RoboSense Airy hemispherical 3D LiDARs.
-  The real model is included unchanged; this file only adds the airy links,
-  their fixed joints and (with sim_gazebo) a gpu_lidar per unit. The unit
-  itself is urdf/airy_lidar.xacro's AiryLidar macro, shared with
-  semi_humanoid_v3.urdf.xacro; see that file for the datasheet mapping and the
-  frame convention.
-  Default mounts: back to back on the body column, facing opposite ways, so the
-  two hemispheres together cover the whole sphere around the robot:
-    airy_link       front (x = +0.200, z = 0.92), pitch +90 deg -> dome faces +x
-    airy_back_link  rear  (x = -0.354, z = 0.77), pitch -90 deg -> dome faces -x
-  Move either one with its own _xyz / _rpy args.
+  semi_humanoid_v2_real.urdf.xacro + one RoboSense Airy hemispherical 3D LiDAR.
+  The real model is included unchanged; this file only adds airy_link, its
+  fixed joint and (with sim_gazebo) a gpu_lidar built from the existing
+  Lidar3DSensor macro in gazebo_plugins.xacro.
+  Airy datasheet, and how each line maps onto this model:
+    Dimension         phi60 x H63 mm, <240 g   -> meshes/airy_lidar.stl, mass
+    FOV (H x V)       360 x 90 deg (hemisphere: from the mounting plane
+                      to the dome axis)        -> vertical 0 .. +90 deg
+    Angular res. H    0.4 deg                  -> 900 horizontal samples
+    Lines             192 / 96 / 48            -> airy_vertical_samples (96)
+    Frame rate        10 Hz                    -> update_rate 10
+    Range             blind spot <0.1 m, max 60 m -> range 0.10 .. 60.0
+    Accuracy          +-1 cm                   -> macro noise (stddev 0.01)
+  192 x 900 is ~173k rays per frame, six times the stock 3D LiDAR; on a Jetson
+  96 lines (the datasheet's 96-beam mode) is the default.
+  airy_link frame: origin at the centre of the mounting face, +z along the
+  dome axis (out of the sensor), the mesh occupies z = 0 .. 0.063. The real
+  optical centre is not published, so the sensor sits on the mounting face;
+  the dome is closer than range_min and does not occlude the rays.
+  Default mount: on the front face of the body column (x = 0.195 m) at the
+  stock 3D LiDAR height, dome facing forward (pitch +90 deg), so the field of
+  view is the whole half-space in front of the robot, floor included. Move it
+  with airy_xyz / airy_rpy.
   Args (in addition to those of semi_humanoid_v2_real.urdf.xacro):
-    airy                        add the front sensor (true)
-    airy_xyz, airy_rpy          front mount pose relative to base_link
-    airy_back                   add the rear sensor (true)
-    airy_back_xyz, airy_back_rpy  rear mount pose relative to base_link
-    airy_vertical_samples       192 / 96 / 48 (96), used by both units
-  Topics (sim_gazebo): gz "airy" and "airy_back"; the launch file bridges them
-  to /airy_points and /airy_back_points.
+    airy                    add the sensor (true)
+    airy_xyz, airy_rpy      mount pose relative to base_link
+    airy_vertical_samples   192 / 96 / 48 (96)
 -->
 <robot name="semi_humanoid_v2" xmlns:xacro="http://ros.org/wiki/xacro">
   <xacro:arg name="airy" default="true"/>
-  <xacro:arg name="airy_xyz" default="0.200 0.0 0.92"/>
+  <xacro:arg name="airy_xyz" default="0.100 0.0 0.92"/>
   <xacro:arg name="airy_rpy" default="0.0 1.5707963 0.0"/>
-  <xacro:arg name="airy_back" default="true"/>
-  <xacro:arg name="airy_back_xyz" default="-0.354 0.0 0.77"/>
-  <xacro:arg name="airy_back_rpy" default="0.0 -1.5707963 0.0"/>
   <xacro:arg name="airy_vertical_samples" default="96"/>
   <xacro:include filename="$(find semi_humanoid_v2)/urdf/semi_humanoid_v2_real.urdf.xacro"/>
-  <!-- Must follow the real model: AiryLidar uses Lidar3DSensor, which
-       gazebo_plugins.xacro defines inside that model's sim_gazebo branch. -->
-  <xacro:include filename="$(find semi_humanoid_v2)/urdf/airy_lidar.xacro"/>
   <xacro:if value="$(arg airy)">
-    <xacro:AiryLidar name="airy" xyz="$(arg airy_xyz)" rpy="$(arg airy_rpy)"
-      vertical_samples="$(arg airy_vertical_samples)"/>
-  </xacro:if>
-  <xacro:if value="$(arg airy_back)">
-    <xacro:AiryLidar name="airy_back" xyz="$(arg airy_back_xyz)" rpy="$(arg airy_back_rpy)"
-      vertical_samples="$(arg airy_vertical_samples)"/>
+    <xacro:property name="airy_radius" value="0.030"/>
+    <xacro:property name="airy_height" value="0.063"/>
+    <xacro:property name="airy_mass" value="0.240"/>
+    <material name="airy_black">
+      <color rgba="0.05 0.05 0.06 1.0"/>
+    </material>
+    <joint name="airy_joint" type="fixed">
+      <parent link="base_link"/>
+      <child link="airy_link"/>
+      <origin xyz="$(arg airy_xyz)" rpy="$(arg airy_rpy)"/>
+    </joint>
+    <link name="airy_link">
+      <inertial>
+        <origin xyz="0 0 ${airy_height/2}" rpy="0 0 0"/>
+        <mass value="${airy_mass}"/>
+        <inertia
+          ixx="${airy_mass/12*(3*airy_radius**2 + airy_height**2)}" ixy="0" ixz="0"
+          iyy="${airy_mass/12*(3*airy_radius**2 + airy_height**2)}" iyz="0"
+          izz="${airy_mass/2*airy_radius**2}"/>
+      </inertial>
+      <visual>
+        <origin xyz="0 0 0" rpy="0 0 0"/>
+        <geometry>
+          <mesh filename="package://semi_humanoid_v2/meshes/airy_lidar.stl"/>
+        </geometry>
+        <material name="airy_black"/>
+      </visual>
+      <collision>
+        <origin xyz="0 0 ${airy_height/2}" rpy="0 0 0"/>
+        <geometry><cylinder radius="${airy_radius}" length="${airy_height}"/></geometry>
+      </collision>
+    </link>
+    <xacro:if value="$(arg sim_gazebo)">
+      <xacro:Lidar3DSensor link="airy_link" topic="airy"
+        horizontal_samples="900" vertical_samples="$(arg airy_vertical_samples)"
+        vertical_min="0.0" vertical_max="${radians(90)}"
+        range_min="0.10" range_max="60.0" update_rate="10"/>
+    </xacro:if>
   </xacro:if>
 </robot>

File: src/semi_humanoid_v2/urdf/semi_humanoid_v2_real.urdf.xacro (robot description, xacro)
@@ -4,5 +4,5 @@
   semi_humanoid_v2.urdf.xacro), ported from antbot_openarm_real.urdf.xacro.
   The base is wired like antbot_description/urdf/antbot.xacro: same wheel
-  macros and the calibrated, upside-down 2D LiDAR mounts. Only GNSS and the 3D
+  macros and the calibrated, upside-down 2D LiDAR mounts. GNSS and the 3D
   LiDAR are absent, as on the sim model.
   Only the Gazebo branch exists so far (robot_sensor_gazebo.launch.py): the
@@ -13,5 +13,5 @@
     sim_gazebo             must stay true for now; also read by
                            openarm_v2_lift.xacro for the Gazebo limit margins
-    camera, side_cameras, lidar_3d   simulated sensors
+    camera, side_cameras             simulated sensors
 -->
 <robot name="semi_humanoid_v2" xmlns:xacro="http://ros.org/wiki/xacro">
@@ -19,5 +19,4 @@
   <xacro:arg name="camera" default="false"/>
   <xacro:arg name="side_cameras" default="false"/>
-  <xacro:arg name="lidar_3d" default="false"/>
   <xacro:arg name="calibration_yaml_path" default=""/>
   <xacro:property name="calibration_yaml_path_val" value="$(arg calibration_yaml_path)"/>
@@ -108,14 +107,4 @@
       <xacro:RgbdCameraSensor link="camera_s10_right_link" topic="camera_s10_right"/>
     </xacro:if>
-    <!-- 3D LiDAR at the stock antbot_description mount. This build has no
-         3D LiDAR, and the column, chest and arms block much of its rear field
-         of view; it is here so antbot_gazebo's lidar_3d option works the same
-         way. -->
-    <xacro:if value="$(arg lidar_3d)">
-      <xacro:CalibratedSensors name="lidar_3d"
-        default_xyz="0.225332 0.0 0.707904" default_rpy="0.0 ${radians(10)} 0.0"
-        calibration_key="lidar_3d_extrinsic"/>
-      <xacro:Lidar3DSensor link="lidar_3d_link" topic="lidar_3d"/>
-    </xacro:if>
   </xacro:if>
 </robot>

File: src/semi_humanoid_v2/urdf/semi_humanoid_v3.urdf.xacro (robot description, xacro)
@@ -17,7 +17,8 @@
       semi_humanoid_v2.urdf.xacro they were silently ignored. Positions are
       unchanged; only the orientations and the calibration hook differ.
-    * lidar_3d at the stock ANTBot mount, optional (lidar_3d, default false),
-      as in semi_humanoid_v2_real.urdf.xacro. This build has no such unit;
-      it is here so antbot_gazebo's lidar_3d option behaves the same way.
+    * NO stock 3D LiDAR. The old ANTBot mount at (0.225332, 0, 0.707904) is
+      gone from every model in this package: this build has no such unit, and
+      there it was heavily occluded by the lift rail, the cargo-box roof and
+      the arms. Use the Airys instead.
     * two RoboSense Airy hemispherical 3D LiDARs, optional (airy / airy_back,
       both default false), at the same mounts as semi_humanoid_v2_airy.
@@ -35,7 +36,6 @@
   <xacro:arg name="sim_gazebo" default="true"/>
   <!-- 3D LiDARs, all off by default: a bare launch costs the same as before. -->
-  <xacro:arg name="lidar_3d" default="false"/>
   <xacro:arg name="airy" default="false"/>
-  <xacro:arg name="airy_xyz" default="0.200 0.0 0.92"/>
+  <xacro:arg name="airy_xyz" default="0.150 0.0 1.00"/>
   <xacro:arg name="airy_rpy" default="0.0 1.5707963 0.0"/>
   <xacro:arg name="airy_back" default="false"/>
@@ -132,14 +132,4 @@
       <xacro:RgbdCameraSensor link="camera_s10_right_link" topic="camera_s10_right"/>
     </xacro:if>
-    <!-- 3D LiDAR at the stock antbot_description mount. This build has no
-         3D LiDAR, and the column, chest and arms block much of its rear field
-         of view; it is here so antbot_gazebo's lidar_3d option works the same
-         way. -->
-    <xacro:if value="$(arg lidar_3d)">
-      <xacro:CalibratedSensors name="lidar_3d"
-        default_xyz="0.225332 0.0 0.707904" default_rpy="0.0 ${radians(10)} 0.0"
-        calibration_key="lidar_3d_extrinsic"/>
-      <xacro:Lidar3DSensor link="lidar_3d_link" topic="lidar_3d"/>
-    </xacro:if>
     <xacro:semi_humanoid_v2_ros2_control_gazebo/>
   </xacro:if>
@@ -147,14 +137,34 @@
        after the sim_gazebo branch above: AiryLidar calls Lidar3DSensor, which
        gazebo_plugins.xacro defines there.
-       v3 has NO top crossbar, so the front unit's nearest structure is now the
-       60x60 lift rail (x 0.070..0.130), 70 mm behind its mounting face; the
-       rear unit still sits flush on the cargo box rear panel (x = -0.354).
-       The two hemispheres do NOT cover the sphere. Each unit sees only its own
-       +X half-space, and the mounts are 0.554 m apart in x, so nothing sees
-       -0.354 < x < 0.200 - a vertical slab through the mid-body, unbounded in
-       y and z. Everything abeam of the robot's middle is invisible to both,
-       which is also where the side S10s have their 0.550 m ceiling. Kept as
-       documented in SENSORS.md; move the mounts onto a shared x plane with the
-       _xyz args if you need the slab closed. -->
+       FRONT unit, (0.150, 0, 1.00), dome facing +X. v3 has no top crossbar,
+       so the 60x60 lift rail is the only structure near it: the rail spans
+       x 0.070..0.130 and z 0.379..1.065, so the mounting face sits 20 mm
+       ahead of the rail's front face and 65 mm BELOW its top - alongside the
+       rail, not above it, which a short bracket off the rail front face
+       reaches. The body occupies x 0.150..0.213 along the dome axis, y +-0.030
+       and z 0.970..1.030.
+       !! THE CHEST DRIVES THROUGH THIS UNIT AT THE TOP OF THE LIFT STROKE !!
+       openarm_lift_link's collision box is x 0.015..0.165, y +-0.080,
+       z (0.730+q)..(0.890+q). Its x and y always overlap the unit; the z bands
+       meet once q >= +0.080, so the whole top 80 mm of the stroke
+       (q = +0.080 .. +0.160) puts the chest 15 mm into the Airy body. At the
+       Gazebo stop (q = +0.165) the overlap is 15 mm in x, 60 mm in y, 60 mm
+       in z. Self-collision is off in the SDF, so nothing stops it - the chest
+       simply passes through, and the unit's own returns will include it.
+       Three ways out, cheapest first: move the mount to x >= 0.165 (just past
+       the chest's front face), or back up to z >= 1.085 (clears the chest's
+       1.055 top at the stop), or cap the lift at q = +0.080. The shoulder
+       crossbar itself is clear either way: x 0.080..0.120, |y| 0.070..0.245,
+       so it misses the unit in both x (30 mm) and y.
+       REAR unit, (-0.354, 0, 0.770), unchanged - flush on the cargo box rear
+       panel, at its top edge.
+       The two hemispheres still do NOT cover the sphere. Each unit sees only
+       its own +X half-space, and the mounts are 0.504 m apart in x, so nothing
+       sees -0.354 < x < 0.150 - a vertical slab through the mid-body,
+       unbounded in y and z. Moving the front unit from 0.200 to 0.150 narrowed
+       that slab by 50 mm but did not close it; everything abeam of the robot's
+       middle is still invisible to both, which is also where the side S10s
+       have their 0.550 m ceiling. Closing it needs both mounts on a shared x
+       plane - set the _xyz args if you want that. -->
   <xacro:if value="$(arg airy)">
     <xacro:AiryLidar name="airy" xyz="$(arg airy_xyz)" rpy="$(arg airy_rpy)"
